File: discipad-pcb.sch (KiCad schematic (older format))
At the start: 56 parts, among them J1 AVR-ISP-6, SW0 KEYSW, SW1 KEYSW, SW10 KEYSW, SW11 KEYSW, SW12 KEYSW, SW13 KEYSW, SW14 KEYSW, SW15 KEYSW, SW16 KEYSW, SW2 KEYSW, SW3 KEYSW, SW4 KEYSW, SW5 KEYSW, SW6 KEYSW, SW7 KEYSW, SW8 KEYSW, SW9 KEYSW, U1 ATmega328P-PU, Y1 Crystal

Commit message: Update discipad-pcb.sch
Parts:
- BOOT1, RESET1: symbol keyboard_parts:SW_PUSH -> discipad-pcb-rescue:SW_PUSH-keyboard_parts
- F1: value 100mA -> 500mA
- J1: symbol Connector:AVR-ISP-6 -> discipad-pcb-rescue:AVR-ISP-6-Connector
- U1: symbol MCU_Microchip_ATmega:ATmega328P-PU -> discipad-pcb-rescue:ATmega328P-PU-MCU_Microchip_ATmega
Other:
- note added: "ISP"
- note added: "MCU"
- note added: "POWER LED"
- note added: "USB/FUSE"
- moved on the sheet: C1, C2, C3, C4, C5, D1, D10, D11, D12, D13, D14, D15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
